File: kicad/power_supply.kicad_sch (KiCad schematic)
At the start: 14 parts, among them U3 LMR38010

Commit message: changes done by jc-efactory: capacitor integrated, a 10mm SMD electrolitic footprint to test fix for issue #68, update to Kicad V9, rerouting, like the 3V3 plane was removed, now a GND layer as well and had to change a couple of capacitor to be able to fit the changes without any major redesign.
Parts:
- C17, C18: footprint LibreSolar:C_1210_3225 -> LibreSolar:C_1206_3216; PartNumber CL32B476MPJNNNE -> CL31A476MPHNNNE
- C22, C23: footprint LibreSolar:C_1210_3225 -> LibreSolar:C_1206_3216; PartNumber CL32B225KCJSNNE -> CL31B225KCHSNNE
Changed lines of the file:
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@@
 (kicad_sch
-	(version 20231120)
+	(version 20250114)
 	(generator "eeschema")
-	(generator_version "8.0")
+	(generator_version "9.0")
 	(paper "A4")
 	(title_block
@@
 		(comment 3 "License: CERN-OHL-W")
 	)
+	(text "ESP32-C3 requires power supply with at least 500 mA"
+		(exclude_from_sim no)
+		(at 129.54 44.45 0)
+		(effects
+			(font
+				(size 1.27 1.27)
+			)
+			(justify left bottom)
+		)
+	)
+	(text "Layout for 500 kHz, 1A output"
+		(exclude_from_sim no)
+		(at 129.54 114.3 0)
+		(effects
+			(font
+				(size 1.27 1.27)
+			)
+			(justify left bottom)
+		)
+	)
+	(text "Battery to 3.3V (SMPS)"
+		(exclude_from_sim no)
+		(at 129.54 38.1 0)
+		(effects
+			(font
+				(size 2.54 2.54)
+			)
+			(justify left bottom)
+		)
+	)
+	(text "Vref = 1.0V"
+		(exclude_from_sim no)
+		(at 172.72 93.98 0)
+		(effects
+			(font
+				(size 1.27 1.27)
+			)
+			(justify left bottom)
+		)
+	)
 	(junction
 		(at 149.86 96.52)
@@
 		)
 	)
-	(text "ESP32-C3 requires power supply with at least 500 mA"
-		(exclude_from_sim no)
-		(at 129.54 44.45 0)
+	(label "SW"
+		(at 165.1 81.28 0)
 		(effects
 			(font
@@
 		)
 	)
-	(text "Layout for 500 kHz, 1A output"
-		(exclude_from_sim no)
-		(at 129.54 114.3 0)
+	(label "VIN"
+		(at 124.46 76.2 0)
 		(effects
 			(font
@@
 		)
 	)
-	(text "Battery to 3.3V (SMPS)"
-		(exclude_from_sim no)
-		(at 129.54 38.1 0)
-		(effects
-			(font
-				(size 2.54 2.54)
-			)
-			(justify left bottom)
-		)
-	)
-	(text "Vref = 1.0V"
-		(exclude_from_sim no)
-		(at 172.72 93.98 0)
+	(label "FB"
+		(at 165.1 88.9 0)
 		(effects
 			(font
@@
 		)
 	)
-	(label "SW"
-		(at 165.1 81.28 0)
-		(fields_autoplaced yes)
+	(hierarchical_label "EN"
+		(shape input)
+		(at 124.46 81.28 180)
 		(effects
 			(font
 				(size 1.27 1.27)
 			)
-			(justify left bottom)
-		)
-	)
-	(label "VIN"
-		(at 124.46 76.2 0)
-		(fields_autoplaced yes)
-		(effects
-			(font
-				(size 1.27 1.27)
-			)
-			(justify left bottom)
-		)
-	)
-	(label "FB"
-		(at 165.1 88.9 0)
-		(fields_autoplaced yes)
-		(effects
-			(font
-				(size 1.27 1.27)
-			)
-			(justify left bottom)
-		)
-	)
-	(hierarchical_label "EN"
-		(shape input)
-		(at 124.46 81.28 180)
-		(fields_autoplaced yes)
-		(effects
-			(font
-				(size 1.27 1.27)
-			)
 			(justify right)
 		)
@@
 		(shape input)
 		(at 63.5 76.2 180)
-		(fields_autoplaced yes)
 		(effects
 			(font
@@
 			)
 		)
-		(property "Footprint" "LibreSolar:C_1210_3225"
+		(property "Footprint" "LibreSolar:C_1206_3216"
 			(at 210.82 93.98 0)
 			(effects
@@
 			)
 		)
-		(property "PartNumber" "CL32B476MPJNNNE"
+		(property "PartNumber" "CL31A476MPHNNNE"
 			(at 45.72 166.37 0)
 			(effects
@@
 			)
 		)
-		(property "Footprint" "LibreSolar:C_1210_3225"
+		(property "Footprint" "LibreSolar:C_1206_3216"
 			(at 200.66 93.98 0)
 			(effects
@@
 			)
 		)
-		(property "PartNumber" "CL32B476MPJNNNE"
+		(property "PartNumber" "CL31A476MPHNNNE"
 			(at 45.72 166.37 0)
 			(effects
@@
 			)
 		)
-		(property "Footprint" "LibreSolar:C_1210_3225"
+		(property "Footprint" "LibreSolar:C_1206_3216"
 			(at 96.52 88.9 0)
 			(effects
@@
 			)
 		)
-		(property "PartNumber" "CL32B225KCJSNNE"
+		(property "PartNumber" "CL31B225KCHSNNE"
 			(at 96.52 83.82 0)
 			(effects
@@
 			)
 		)
-		(property "Footprint" "LibreSolar:C_1210_3225"
+		(property "Footprint" "LibreSolar:C_1206_3216"
 			(at 86.36 88.9 0)
 			(effects
@@
 			)
 		)
-		(property "PartNumber" "CL32B225KCJSNNE"
+		(property "PartNumber" "CL31B225KCHSNNE"
 			(at 10.16 153.67 0)
 			(effects
